Commit message: Improve live Gazebo ROSbot security scenarios
Import pinned manufacturer models and render measured product joints. Add walking person reports, manual scene progression and secured Gazebo attack probes. Fix world-triggered stop progression and retain terminal errors in the live viewer. Update runbooks, continuation notes and regression checks while excluding local runtime and advisor artifacts.

File: ros/gazebo/reference_bot.urdf.xacro (robot description, xacro)
@@ -1,8 +1,14 @@
 <?xml version="1.0"?>
-<!-- Small mobile manipulator for Gazebo Harmonic. Geometry is illustrative. -->
+<!-- Small mobile manipulator for Gazebo Harmonic. The visual shell is illustrative. -->
 <robot name="haetae_reference" xmlns:xacro="http://www.ros.org/wiki/xacro">
   <xacro:arg name="controllers_file" default=""/>
+  <xacro:arg name="meshes_dir" default="/workspace/ros/gazebo/meshes"/>
+  <material name="graphite"><color rgba="0.10 0.16 0.21 1"/></material>
+  <material name="shell_white"><color rgba="0.88 0.94 0.95 1"/></material>
+  <material name="sensor_glass"><color rgba="0.035 0.09 0.13 1"/></material>
+  <material name="sensor_teal"><color rgba="0.13 0.75 0.78 1"/></material>
+  <material name="arm_silver"><color rgba="0.61 0.72 0.76 1"/></material>
   <link name="chassis">
-    <visual><origin xyz="0 0 0.20"/><geometry><box size="0.40 0.30 0.20"/></geometry></visual>
+    <visual name="authored_shell"><geometry><mesh filename="file://$(arg meshes_dir)/chassis.dae"/></geometry></visual>
     <collision><origin xyz="0 0 0.20"/><geometry><box size="0.40 0.30 0.20"/></geometry></collision>
     <inertial><origin xyz="0 0 0.20"/><mass value="4"/><inertia ixx="0.05" ixy="0" ixz="0" iyy="0.08" iyz="0" izz="0.08"/></inertial>
@@ -10,5 +16,5 @@
   <xacro:macro name="wheel" params="side y">
     <link name="${side}_wheel">
-      <visual><geometry><cylinder radius="0.10" length="0.04"/></geometry></visual>
+    <visual name="authored_shell"><geometry><mesh filename="file://$(arg meshes_dir)/wheel.dae"/></geometry></visual>
       <collision><geometry><cylinder radius="0.10" length="0.04"/></geometry></collision>
       <inertial><mass value="0.25"/><inertia ixx="0.001" ixy="0" ixz="0" iyy="0.001" iyz="0" izz="0.001"/></inertial>
@@ -23,5 +29,5 @@
   <xacro:wheel side="right" y="-0.18"/>
   <link name="caster">
-    <visual><geometry><sphere radius="0.05"/></geometry></visual>
+    <visual><geometry><sphere radius="0.05"/></geometry><material name="graphite"/></visual>
     <collision><geometry><sphere radius="0.05"/></geometry></collision>
     <inertial><mass value="0.05"/><inertia ixx="0.0001" ixy="0" ixz="0" iyy="0.0001" iyz="0" izz="0.0001"/></inertial>
@@ -31,5 +37,5 @@
   </joint>
   <link name="arm">
-    <visual><origin xyz="0.15 0 0"/><geometry><box size="0.30 0.04 0.04"/></geometry></visual>
+    <visual name="authored_shell"><geometry><mesh filename="file://$(arg meshes_dir)/arm.dae"/></geometry></visual>
     <collision><origin xyz="0.15 0 0"/><geometry><box size="0.30 0.04 0.04"/></geometry></collision>
     <inertial><origin xyz="0.15 0 0"/><mass value="0.2"/><inertia ixx="0.0001" ixy="0" ixz="0" iyy="0.002" iyz="0" izz="0.002"/></inertial>
